Commit message: changed mk-1

File: tonian/assets/urdf/mk-1/robot.urdf (robot description, URDF)
Before this commit: robot onshape, 18 links, 17 joints
Links:
- added link torso, mass 1e-9
Joints:
- added joint torso_frame: type fixed, parent upper_torso, child torso, origin xyz=0.637598 -0.133456 2.05183 rpy=-1.5708 -0 1.38778e-16, axis 0 0 0
- joint left_elbow: origin xyz=4.44089e-16 -1.38778e-17 -0.38 rpy=1.5708 6.20142e-30 1.5708 -> xyz=0 -1.38778e-17 -0.38 rpy=1.5708 6.20142e-30 1.5708
- joint left_foot: origin xyz=0.02 0.53 -2.22045e-16 rpy=3.14159 -1.97232e-14 3.10995 -> xyz=0.02 0.53 0 rpy=-3.14159 -4.77009e-15 -3.12934
- joint left_hip_a: child lower_torso -> torso_leg_connector; limit lower=-0.349066 upper=0.349066 effort=1 velocity=20 -> lower=-0.523599 upper=0.523599 effort=1 velocity=20; origin xyz=0.712598 0.0214372 1.31464 rpy=-2.49096e-23 1.04618e-22 3.14017 -> xyz=-0.075 -1.38778e-17 -0.07 rpy=3.14159 -3.3777e-20 -1.53511; parent torso_leg_connector -> lower_torso
- joint left_hip_b: limit lower=-1.74533 upper=0 effort=1 velocity=20 -> lower=0 upper=1.74533 effort=1 velocity=20; origin xyz=0.840594 0.0204162 1.31463 rpy=-1.5708 -0.0224217 -1.57877 -> xyz=0 0.128 -3.2634e-06 rpy=1.5708 -0.0128273 3.33077e-16
- joint left_knee: limit lower=-1.91986 upper=0 effort=1 velocity=20 -> lower=-1.5708 upper=0 effort=1 velocity=20; origin xyz=2.44162e-16 0.5 2.22045e-16 rpy=-3.14159 -1.61144e-15 -3.14159 -> xyz=3.46945e-18 0.5 0 rpy=-1.09538e-21 -4.34006e-22 -4.02109e-16
- joint left_shoulder_a: origin xyz=0.193521 0.0155608 -0.786479 rpy=0.785398 1.58051e-14 -1.5708 -> xyz=0.83112 0.00598303 2.17112 rpy=-2.35619 -1.58051e-14 1.5708
- joint right_foot: origin xyz=0.02 -0.53 -1.11022e-16 rpy=1.6217e-15 -1.50899e-14 -3.10906 -> xyz=0.02 -0.53 0 rpy=1.57718e-15 -1.4282e-14 -3.10904
- joint right_hip_a: origin xyz=0.15 9.54445e-15 0 rpy=-3.14159 -6.12323e-17 1.61306 -> xyz=0.075 2.22045e-16 -0.07 rpy=-3.14159 3.62558e-19 1.61597
- joint right_hip_b: origin xyz=3.90313e-18 0.128 -3.2634e-06 rpy=1.5708 0.0235009 2.26335e-15 -> xyz=-6.93889e-18 0.128 -3.2634e-06 rpy=1.5708 0.0235125 1.4408e-15
- joint right_knee: origin xyz=6.93889e-18 0.5 0 rpy=-1.93571e-15 1.78614e-15 3.14159 -> xyz=-1.73472e-18 0.5 0 rpy=-1.94365e-15 1.84117e-15 3.14159
- joint right_shoulder_a: origin xyz=-0.193521 0.0155608 -0.786479 rpy=-0.785398 -4.62008e-14 -1.5708 -> xyz=0.444077 0.00598303 2.17112 rpy=2.35619 4.62008e-14 1.5708
- joint torso: child upper_torso -> lower_torso; origin xyz=0.075 1.04083e-17 0.07 rpy=3.14159 1.04653e-22 -3.14017 -> xyz=0.637598 0.0215438 1.38464 rpy=3.17888e-20 7.51828e-21 3.1059; parent lower_torso -> upper_torso

Commit message: fixed the misplaced axis issue

File: tonian/assets/urdf/mk-1/robot.urdf (robot description, URDF)
Before this commit: robot onshape, 19 links, 18 joints
Joints:
- joint left_arm_rotate: origin xyz=-0.102112 0.170673 -1.38778e-17 rpy=-1.5708 5.64975e-15 -3.14159 -> xyz=-0.102112 0.170673 -2.08167e-17 rpy=-1.5708 5.64975e-15 -3.14159
- joint left_elbow: origin xyz=0 -1.38778e-17 -0.38 rpy=1.5708 6.20142e-30 1.5708 -> xyz=-1.11022e-16 -2.08167e-17 -0.38 rpy=1.5708 6.20142e-30 1.5708
- joint left_foot: origin xyz=0.02 0.53 0 rpy=-3.14159 -4.77009e-15 -3.12934 -> xyz=0.02 0.53 -8.32667e-17 rpy=-3.14159 -4.77009e-15 -3.12934
- joint left_hip_a: origin xyz=-0.075 -1.38778e-17 -0.07 rpy=3.14159 -3.3777e-20 -1.53511 -> xyz=-0.075 -2.08167e-17 -0.07 rpy=3.14159 -3.3777e-20 -1.53511
- joint left_hip_b: origin xyz=0 0.128 -3.2634e-06 rpy=1.5708 -0.0128273 3.33077e-16 -> xyz=-3.46945e-18 0.128 -3.2634e-06 rpy=1.5708 -0.0128273 3.33077e-16
- joint left_knee: origin xyz=3.46945e-18 0.5 0 rpy=-1.09538e-21 -4.34006e-22 -4.02109e-16 -> xyz=0 0.5 0 rpy=-1.09538e-21 -4.34006e-22 -4.02109e-16
- joint left_shoulder_a: origin xyz=0.83112 0.00598303 2.17112 rpy=-2.35619 -1.58051e-14 1.5708 -> xyz=0.193731 -0.0416859 0.390756 rpy=-2.35619 -1.58051e-14 1.5708
- joint right_arm_rotate: origin xyz=-0.102112 0.170673 -5.9848e-17 rpy=1.5708 -3.80147e-17 2.34892e-16 -> xyz=-0.102112 0.170673 -2.08167e-17 rpy=1.5708 -3.80147e-17 2.34892e-16
- joint right_elbow: origin xyz=4.44089e-16 -2.1684e-17 -0.38 rpy=1.5708 -3.86634e-30 1.5708 -> xyz=1.11022e-16 -2.08167e-17 -0.38 rpy=1.5708 -3.86634e-30 1.5708
- joint right_foot: origin xyz=0.02 -0.53 0 rpy=1.57718e-15 -1.4282e-14 -3.10904 -> xyz=0.02 -0.53 -8.32667e-17 rpy=1.57718e-15 -1.4282e-14 -3.10904
- joint right_hip_a: origin xyz=0.075 2.22045e-16 -0.07 rpy=-3.14159 3.62558e-19 1.61597 -> xyz=0.075 -2.08167e-17 -0.07 rpy=-3.14159 3.62558e-19 1.61597
- joint right_hip_b: origin xyz=-6.93889e-18 0.128 -3.2634e-06 rpy=1.5708 0.0235125 1.4408e-15 -> xyz=0 0.128 -3.2634e-06 rpy=1.5708 0.0235125 1.4408e-15
- joint right_shoulder_a: origin xyz=0.444077 0.00598303 2.17112 rpy=2.35619 4.62008e-14 1.5708 -> xyz=-0.193311 -0.0416859 0.390756 rpy=2.35619 4.62008e-14 1.5708
- joint torso: origin xyz=0.637598 0.0215438 1.38464 rpy=3.17888e-20 7.51828e-21 3.1059 -> xyz=0.000209962 -0.0261252 -0.395722 rpy=3.17888e-20 7.51828e-21 3.1059
- joint torso_frame: origin xyz=0.637598 -0.133456 2.05183 rpy=-1.5708 -0 1.38778e-16 -> xyz=0.000209962 -0.181125 0.271472 rpy=-1.5708 -0 1.38778e-16

Commit message: good console outputs

File: tonian/assets/urdf/mk-1/robot.urdf (robot description, URDF)
Before this commit: robot onshape, 19 links, 18 joints
Links:
- link forearm: mass 4.07336 -> 6.10911
- link forearm_2: mass 4.07336 -> 6.10911
Joints:
- joint left_hip_a: origin xyz=-0.075 -2.08167e-17 -0.07 rpy=3.14159 -3.3777e-20 -1.53511 -> xyz=-0.075 -1.73472e-17 -0.07 rpy=3.14159 -3.3777e-20 -1.53511
- joint left_knee: origin xyz=0 0.5 0 rpy=-1.09538e-21 -4.34006e-22 -4.02109e-16 -> xyz=3.46945e-18 0.5 0 rpy=-1.09538e-21 -4.34006e-22 -4.02109e-16
- joint left_shoulder_a: origin xyz=0.193731 -0.0416859 0.390756 rpy=-2.35619 -1.58051e-14 1.5708 -> xyz=0.193731 -0.0416858 0.390756 rpy=-2.35619 -1.58051e-14 1.5708
- joint right_hip_a: origin xyz=0.075 -2.08167e-17 -0.07 rpy=-3.14159 3.62558e-19 1.61597 -> xyz=0.075 -1.73472e-17 -0.07 rpy=-3.14159 3.62558e-19 1.61597
- joint right_knee: origin xyz=-1.73472e-18 0.5 0 rpy=-1.94365e-15 1.84117e-15 3.14159 -> xyz=-3.46945e-18 0.5 -2.77556e-17 rpy=-1.94365e-15 1.84117e-15 3.14159
- joint right_shoulder_a: origin xyz=-0.193311 -0.0416859 0.390756 rpy=2.35619 4.62008e-14 1.5708 -> xyz=-0.193311 -0.0416858 0.390756 rpy=2.35619 4.62008e-14 1.5708
- joint torso: origin xyz=0.000209962 -0.0261252 -0.395722 rpy=3.17888e-20 7.51828e-21 3.1059 -> xyz=0.000209995 -0.0261251 -0.395722 rpy=3.17888e-20 7.51828e-21 3.1059
- joint torso_frame: origin xyz=0.000209962 -0.181125 0.271472 rpy=-1.5708 -0 1.38778e-16 -> xyz=0.000209995 -0.181125 0.271472 rpy=-1.5708 -0 1.38778e-16

Commit message: added scad files and pure shapes approx for mk1

File: tonian/assets/urdf/mk-1/robot.urdf (robot description, URDF)
Before this commit: robot onshape, 19 links, 18 joints
Links:
- link foot: geometry collision box size=0.13 0.3 0.04; visual mesh filename=package://foot.stl
- link foot_2: geometry collision box size=0.13 0.3 0.04; visual mesh filename=package://foot.stl
- link forearm: geometry collision cylinder length=0.11 radius=0.015; collision cylinder length=0.14 radius=0.04
- link forearm_2: geometry collision cylinder length=0.11 radius=0.015; collision cylinder length=0.14 radius=0.04
- link lower_leg: geometry collision box size=0.14 0.43 0.1; collision cylinder length=0.07 radius=0.015
- link lower_leg_2: geometry collision box size=0.14 0.43 0.1; collision cylinder length=0.07 radius=0.015
- link lower_torso: geometry collision box size=0.04 0.2 0.2; visual mesh filename=package://lower_torso.stl
- link shoulder: geometry collision cylinder length=0.1 radius=0.05; visual mesh filename=package://shoulder.stl
- link shoulder-connector: geometry collision cylinder length=0.08 radius=0.05; visual mesh filename=package://shoulder-connector.stl
- link shoulder-connector_2: geometry collision cylinder length=0.08 radius=0.05; visual mesh filename=package://shoulder-connector.stl
- link shoulder_2: geometry collision cylinder length=0.1 radius=0.05; visual mesh filename=package://shoulder.stl
- link torso_leg_connector: geometry collision cylinder length=0.23 radius=0.03; visual mesh filename=package://torso_leg_connector.stl
- link torso_leg_connector_2: geometry collision cylinder length=0.23 radius=0.03; visual mesh filename=package://torso_leg_connector.stl
- link upper_arm: geometry collision cylinder length=0.33 radius=0.05; collision cylinder length=0.42 radius=0.05
- link upper_arm_2: geometry collision cylinder length=0.33 radius=0.05; collision cylinder length=0.42 radius=0.05
- link upper_leg: geometry collision box size=0.14 0.38 0.01; collision box size=0.142368 0.379314 0.01
- link upper_leg_2: geometry collision box size=0.14 0.38 0.01; collision box size=0.142368 0.379314 0.01
- link upper_torso: geometry collision box size=0.270651 0.13 0.2; collision box size=0.4 0.4 0.2
Joints:
- joint left_foot: origin xyz=0.02 0.53 -8.32667e-17 rpy=-3.14159 -4.77009e-15 -3.12934 -> xyz=0.02 0.53 -1.11022e-16 rpy=-3.14159 -4.77009e-15 -3.12934
- joint left_knee: origin xyz=3.46945e-18 0.5 0 rpy=-1.09538e-21 -4.34006e-22 -4.02109e-16 -> xyz=0 0.5 0 rpy=-1.09538e-21 -4.34006e-22 -4.02109e-16
- joint left_shoulder_a: origin xyz=0.193731 -0.0416858 0.390756 rpy=-2.35619 -1.58051e-14 1.5708 -> xyz=0.193732 -0.0416846 0.390757 rpy=-2.35619 -1.58051e-14 1.5708
- joint right_foot: origin xyz=0.02 -0.53 -8.32667e-17 rpy=1.57718e-15 -1.4282e-14 -3.10904 -> xyz=0.02 -0.53 -2.77556e-17 rpy=1.57718e-15 -1.4282e-14 -3.10904
- joint right_knee: origin xyz=-3.46945e-18 0.5 -2.77556e-17 rpy=-1.94365e-15 1.84117e-15 3.14159 -> xyz=0 0.5 2.77556e-17 rpy=-1.94365e-15 1.84117e-15 3.14159
- joint right_shoulder_a: origin xyz=-0.193311 -0.0416858 0.390756 rpy=2.35619 4.62008e-14 1.5708 -> xyz=-0.193311 -0.0416846 0.390757 rpy=2.35619 4.62008e-14 1.5708
- joint torso: origin xyz=0.000209995 -0.0261251 -0.395722 rpy=3.17888e-20 7.51828e-21 3.1059 -> xyz=0.000210489 -0.0261238 -0.395722 rpy=3.17888e-20 7.51828e-21 3.1059
- joint torso_frame: origin xyz=0.000209995 -0.181125 0.271472 rpy=-1.5708 -0 1.38778e-16 -> xyz=0.000210489 -0.181124 0.271473 rpy=-1.5708 -0 1.38778e-16
