Commit message: added shitty cassie

File: tonian/assets/cassie/urdf/cassie.urdf (robot description, URDF)
Before this commit: robot cassie, 18 links, 17 joints
Links:
- link left_hip: geometry collision mesh filename=./../meshes/hip.stl scale=1 1 1; visual mesh filename=./../meshes/hip.stl scale=1 1 1
- link left_knee: geometry collision mesh filename=./../meshes/knee-output.stl scale=1 1 1; visual mesh filename=./../meshes/knee-output.stl scale=1 1 1
- link left_pelvis_abduction: geometry collision mesh filename=./../meshes/abduction.stl scale=1 1 1; visual mesh filename=./../meshes/abduction.stl scale=1 1 1
- link left_pelvis_rotation: geometry collision mesh filename=./../meshes/yaw.stl scale=1 1 1; visual mesh filename=./../meshes/yaw.stl scale=1 1 1
- link left_shin: geometry collision mesh filename=./../meshes/shin-bone.stl scale=1 1 1; visual mesh filename=./../meshes/shin-bone.stl scale=1 1 1
- link left_tarsus: geometry collision mesh filename=./../meshes/tarsus.stl scale=1 1 1; visual mesh filename=./../meshes/tarsus.stl scale=1 1 1
- link left_thigh: geometry collision mesh filename=./../meshes/thigh.stl scale=1 1 1; visual mesh filename=./../meshes/thigh.stl scale=1 1 1
- link left_toe: geometry collision mesh filename=./../meshes/toe.stl scale=1 1 1; visual mesh filename=./../meshes/toe.stl scale=1 1 1
- link pelvis: geometry collision mesh filename=./../meshes/pelvis.stl scale=1 1 1; visual mesh filename=./../meshes/pelvis.stl scale=1 1 1
- link right_hip: geometry collision mesh filename=./../meshes/hip_mirror.stl scale=1 1 1; visual mesh filename=./../meshes/hip_mirror.stl scale=1 1 1
- link right_knee: geometry collision mesh filename=./../meshes/knee-output_mirror.stl scale=1 1 1; visual mesh filename=./../meshes/knee-output_mirror.stl scale=1 1 1
- link right_pelvis_abduction: geometry collision mesh filename=./../meshes/abduction_mirror.stl scale=1 1 1; visual mesh filename=./../meshes/abduction_mirror.stl scale=1 1 1
- link right_pelvis_rotation: geometry collision mesh filename=./../meshes/yaw_mirror.stl scale=1 1 1; visual mesh filename=./../meshes/yaw_mirror.stl scale=1 1 1
- link right_shin: geometry collision mesh filename=./../meshes/shin-bone_mirror.stl scale=1 1 1; visual mesh filename=./../meshes/shin-bone_mirror.stl scale=1 1 1
- link right_tarsus: geometry collision mesh filename=./../meshes/tarsus_mirror.stl scale=1 1 1; visual mesh filename=./../meshes/tarsus_mirror.stl scale=1 1 1
- link right_thigh: geometry collision mesh filename=./../meshes/thigh_mirror.stl scale=1 1 1; visual mesh filename=./../meshes/thigh_mirror.stl scale=1 1 1
- link right_toe: geometry collision mesh filename=./../meshes/toe_mirror.stl scale=1 1 1; visual mesh filename=./../meshes/toe_mirror.stl scale=1 1 1

File: tonian/assets/cassie/urdf/cassie_with_base.urdf (robot description, URDF)
Before this commit: robot cassie, 24 links, 23 joints
Links:
- link left_hip: geometry visual mesh filename=./../meshes/hip.stl scale=1 1 1
- link left_knee: geometry visual mesh filename=./../meshes/knee-output.stl scale=1 1 1
- link left_pelvis_abduction: geometry visual mesh filename=./../meshes/abduction.stl scale=1 1 1
- link left_pelvis_rotation: geometry visual mesh filename=./../meshes/yaw.stl scale=1 1 1
- link left_shin: geometry visual mesh filename=./../meshes/shin-bone.stl scale=1 1 1
- link left_tarsus: geometry visual mesh filename=./../meshes/tarsus.stl scale=1 1 1
- link left_thigh: geometry visual mesh filename=./../meshes/thigh.stl scale=1 1 1
- link left_toe: geometry visual mesh filename=./../meshes/toe.stl scale=1 1 1
- link pelvis: geometry visual mesh filename=./../meshes/pelvis.stl scale=1 1 1
- link right_hip: geometry visual mesh filename=./../meshes/hip_mirror.stl scale=1 1 1
- link right_knee: geometry visual mesh filename=./../meshes/knee-output_mirror.stl scale=1 1 1
- link right_pelvis_abduction: geometry visual mesh filename=./../meshes/abduction_mirror.stl scale=1 1 1
- link right_pelvis_rotation: geometry visual mesh filename=./../meshes/yaw_mirror.stl scale=1 1 1
- link right_shin: geometry visual mesh filename=./../meshes/shin-bone_mirror.stl scale=1 1 1
- link right_tarsus: geometry visual mesh filename=./../meshes/tarsus_mirror.stl scale=1 1 1
- link right_thigh: geometry visual mesh filename=./../meshes/thigh_mirror.stl scale=1 1 1
- link right_toe: geometry visual mesh filename=./../meshes/toe_mirror.stl scale=1 1 1

File: tonian/assets/cassie/urdf/cassie_with_torso.urdf (robot description, URDF)
Before this commit: robot cassie, 23 links, 22 joints
Links:
- link left_hip: geometry visual mesh filename=./../meshes/hip.stl scale=1 1 1
- link left_knee: geometry visual mesh filename=./../meshes/knee-output.stl scale=1 1 1
- link left_pelvis_abduction: geometry visual mesh filename=./../meshes/abduction.stl scale=1 1 1
- link left_pelvis_rotation: geometry visual mesh filename=./../meshes/yaw.stl scale=1 1 1
- link left_shin: geometry visual mesh filename=./../meshes/shin-bone.stl scale=1 1 1
- link left_tarsus: geometry visual mesh filename=./../meshes/tarsus.stl scale=1 1 1
- link left_thigh: geometry visual mesh filename=./../meshes/thigh.stl scale=1 1 1
- link left_toe: geometry visual mesh filename=./../meshes/toe.stl scale=1 1 1
- link pelvis: geometry visual mesh filename=./../meshes/pelvis.stl scale=1 1 1
- link right_hip: geometry visual mesh filename=./../meshes/hip_mirror.stl scale=1 1 1
- link right_knee: geometry visual mesh filename=./../meshes/knee-output_mirror.stl scale=1 1 1
- link right_pelvis_abduction: geometry visual mesh filename=./../meshes/abduction_mirror.stl scale=1 1 1
- link right_pelvis_rotation: geometry visual mesh filename=./../meshes/yaw_mirror.stl scale=1 1 1
- link right_shin: geometry visual mesh filename=./../meshes/shin-bone_mirror.stl scale=1 1 1
- link right_tarsus: geometry visual mesh filename=./../meshes/tarsus_mirror.stl scale=1 1 1
- link right_thigh: geometry visual mesh filename=./../meshes/thigh_mirror.stl scale=1 1 1
- link right_toe: geometry visual mesh filename=./../meshes/toe_mirror.stl scale=1 1 1
- link torso: geometry visual mesh filename=./../meshes/torso.stl scale=1 1 1

File: tonian/assets/cassie/urdf/robot.urdf (robot description, URDF)
Before this commit: robot cassie, 18 links, 17 joints
Links:
- link left_hip: geometry visual mesh filename=./../meshes/hip.stl scale=1 1 1
- link left_knee: geometry visual mesh filename=./../meshes/knee-output.stl scale=1 1 1
- link left_pelvis_abduction: geometry visual mesh filename=./../meshes/abduction.stl scale=1 1 1
- link left_pelvis_rotation: geometry visual mesh filename=./../meshes/yaw.stl scale=1 1 1
- link left_shin: geometry visual mesh filename=./../meshes/shin-bone.stl scale=1 1 1
- link left_tarsus: geometry visual mesh filename=./../meshes/tarsus.stl scale=1 1 1
- link left_thigh: geometry visual mesh filename=./../meshes/thigh.stl scale=1 1 1
- link left_toe: geometry visual mesh filename=./../meshes/toe.stl scale=1 1 1
- link pelvis: geometry visual mesh filename=./../meshes/pelvis.stl scale=1 1 1
- link right_hip: geometry visual mesh filename=./../meshes/hip_mirror.stl scale=1 1 1
- link right_knee: geometry visual mesh filename=./../meshes/knee-output_mirror.stl scale=1 1 1
- link right_pelvis_abduction: geometry visual mesh filename=./../meshes/abduction_mirror.stl scale=1 1 1
- link right_pelvis_rotation: geometry visual mesh filename=./../meshes/yaw_mirror.stl scale=1 1 1
- link right_shin: geometry visual mesh filename=./../meshes/shin-bone_mirror.stl scale=1 1 1
- link right_tarsus: geometry visual mesh filename=./../meshes/tarsus_mirror.stl scale=1 1 1
- link right_thigh: geometry visual mesh filename=./../meshes/thigh_mirror.stl scale=1 1 1
- link right_toe: geometry visual mesh filename=./../meshes/toe_mirror.stl scale=1 1 1

File: tonian/assets/cassie/urdf/torso.urdf (robot description, URDF)
Before this commit: robot cassie, 5 links, 4 joints
Links:
- link torso: geometry visual mesh filename=./../meshes/torso.stl scale=1 1 1
